File: scripts/irrigazione/kicad/irrigazione.sch (KiCad schematic (older format))
At the start: 13 parts

Commit message: Modificha ai condensatori, export svg
Parts:
- removed C? (x2): CP, symbol CP
- added C1: 10nF, symbol CP_Small
- added C2: 10uF, symbol CP_Small
- gave numbers to parts that had none: 11
Connections:
- wire segments 49 -> 59
Changed lines of the file:
@@
 $EndDescr
 $Comp
-L TRANSFO T?
+L TRANSFO T1
 U 1 1 55144E98
 P 6520 3510
-F 0 "T?" H 6570 3560 60  0001 C CNN
+F 0 "T1" H 6570 3560 60  0001 C CNN
 F 1 "TRANSFO" H 6520 3510 60  0001 C CNN
 F 2 "" H 6520 3510 60  0001 C CNN
@@
 $EndComp
 $Comp
-L TLP185 U?
+L TLP185 U3
 U 1 1 55145077
 P 4470 4210
-F 0 "U?" H 4520 4260 60  0001 C CNN
+F 0 "U3" H 4520 4260 60  0001 C CNN
 F 1 "TLP185" H 4470 4210 60  0001 C CNN
 F 2 "" H 4470 4210 60  0001 C CNN
@@
 $EndComp
 $Comp
-L TLP185 U?
+L TLP185 U4
 U 1 1 55145097
 P 7670 4210
-F 0 "U?" H 7720 4260 60  0001 C CNN
+F 0 "U4" H 7720 4260 60  0001 C CNN
 F 1 "TLP185" H 7670 4210 60  0001 C CNN
 F 2 "" H 7670 4210 60  0001 C CNN
@@
 $EndComp
 $Comp
-L RM50-xx11 RL?
+L RM50-xx11 RL1
 U 1 1 55145121
 P 5270 3410
-F 0 "RL?" H 5320 3460 60  0001 C CNN
+F 0 "RL1" H 5320 3460 60  0001 C CNN
 F 1 "RM50-xx11" H 5270 3410 60  0001 C CNN
 F 2 "" H 5270 3410 60  0001 C CNN
@@
 $EndComp
 $Comp
-L RM50-xx11 RL?
+L RM50-xx11 RL2
 U 1 1 55145141
 P 8470 3110
-F 0 "RL?" H 8520 3160 60  0001 C CNN
+F 0 "RL2" H 8520 3160 60  0001 C CNN
 F 1 "RM50-xx11" H 8470 3110 60  0001 C CNN
 F 2 "" H 8470 3110 60  0001 C CNN
@@
 	4970 3210 4770 3210
 Wire Wire Line
-	4770 2760 4770 4110
+	4770 2760 4770 3210
+Wire Wire Line
+	4770 3210 4770 4110
 Wire Wire Line
 	8170 2910 7970 2910
 Wire Wire Line
-	7970 2460 7970 4110
-$Comp
-L GND #PWR?
+	7970 2460 7970 2910
+Wire Wire Line
+	7970 2910 7970 4110
+$Comp
+L GND #PWR4
 U 1 1 55145278
 P 4770 4610
-F 0 "#PWR?" H 4820 4660 60  0001 C CNN
+F 0 "#PWR4" H 4820 4660 60  0001 C CNN
 F 1 "GND" H 4770 4610 60  0001 C CNN
 F 2 "" H 4770 4610 60  0001 C CNN
@@
 $EndComp
 $Comp
-L GND #PWR?
+L GND #PWR9
 U 1 1 55145298
 P 7970 4610
-F 0 "#PWR?" H 8020 4660 60  0001 C CNN
+F 0 "#PWR9" H 8020 4660 60  0001 C CNN
 F 1 "GND" H 7970 4610 60  0001 C CNN
 F 2 "" H 7970 4610 60  0001 C CNN
@@
 	4770 4310 4770 4610
 $Comp
-L VCC #PWR?
+L VCC #PWR5
 U 1 1 551452C5
 P 5570 2710
-F 0 "#PWR?" H 5620 2760 60  0001 C CNN
+F 0 "#PWR5" H 5620 2760 60  0001 C CNN
 F 1 "VCC" H 5570 2710 60  0001 C CNN
 F 2 "" H 5570 2710 60  0001 C CNN
@@
 $EndComp
 Wire Wire Line
-	5570 2710 5570 3210
-$Comp
-L VCC #PWR?
+	5570 2710 5570 2760
+Wire Wire Line
+	5570 2760 5570 3210
+$Comp
+L VCC #PWR10
 U 1 1 551452ED
 P 8770 2410
-F 0 "#PWR?" H 8820 2460 60  0001 C CNN
+F 0 "#PWR10" H 8820 2460 60  0001 C CNN
 F 1 "VCC" H 8770 2410 60  0001 C CNN
 F 2 "" H 8770 2410 60  0001 C CNN
@@
 $EndComp
 Wire Wire Line
-	8770 2410 8770 2910
-$Comp
-L D D?
+	8770 2410 8770 2460
+Wire Wire Line
+	8770 2460 8770 2910
+$Comp
+L D D2
 U 1 1 55145316
 P 8470 2460
-F 0 "D?" H 8520 2510 60  0001 C CNN
+F 0 "D2" H 8520 2510 60  0001 C CNN
 F 1 "D" H 8470 2460 60  0001 C CNN
 F 2 "" H 8470 2460 60  0001 C CNN
@@
 Connection ~ 7970 2910
 $Comp
-L D D?
+L D D1
 U 1 1 55145350
 P 5270 2760
-F 0 "D?" H 5320 2810 60  0001 C CNN
+F 0 "D1" H 5320 2810 60  0001 C CNN
 F 1 "D" H 5270 2760 60  0001 C CNN
 F 2 "" H 5270 2760 60  0001 C CNN
@@
 	5570 3710 6120 3710
 $Comp
-L VSS #PWR?
+L VSS #PWR6
 U 1 1 551453A6
 P 5720 2160
-F 0 "#PWR?" H 5770 2210 60  0001 C CNN
+F 0 "#PWR6" H 5770 2210 60  0001 C CNN
 F 1 "VSS" H 5720 2160 60  0001 C CNN
 F 2 "" H 5720 2160 60  0001 C CNN
@@
 $EndComp
 $Comp
-L VSS #PWR?
+L VSS #PWR7
 U 1 1 551453C6
 P 6020 2160
-F 0 "#PWR?" H 6070 2210 60  0001 C CNN
+F 0 "#PWR7" H 6070 2210 60  0001 C CNN
 F 1 "VSS" H 6020 2160 60  0001 C CNN
 F 2 "" H 6020 2160 60  0001 C CNN
@@
 	6920 3310 8170 3310
 $Comp
-L INDUCTOR L?
+L INDUCTOR L1
 U 1 1 5514542A
 P 9820 3210
-F 0 "L?" H 9870 3260 60  0001 C CNN
+F 0 "L1" H 9870 3260 60  0001 C CNN
 F 1 "INDUCTOR" H 9820 3210 60  0001 C CNN
 F 2 "" H 9820 3210 60  0001 C CNN
@@
 $EndComp
 $Comp
-L INDUCTOR L?
+L INDUCTOR L2
 U 1 1 5514544A
 P 9820 3410
-F 0 "L?" H 9870 3460 60  0001 C CNN
+F 0 "L2" H 9870 3460 60  0001 C CNN
 F 1 "INDUCTOR" H 9820 3410 60  0001 C CNN
 F 2 "" H 9820 3410 60  0001 C CNN
@@
 	10070 3210 10170 3210
 Wire Wire Line
-	10170 3210 10170 3710
+	10170 3210 10170 3410
+Wire Wire Line
+	10170 3410 10170 3710
 Wire Wire Line
 	10170 3710 6920 3710
@@
 Connection ~ 10170 3410
 $Comp
-L ESP8266-ESP-01 U?
+L ESP8266-ESP-01 U2
 U 1 1 551455B6
 P 3420 3160
-F 0 "U?" H 3470 3210 60  0001 C CNN
+F 0 "U2" H 3470 3210 60  0001 C CNN
 F 1 "ESP8266-ESP-01" H 3420 3160 60  0001 C CNN
 F 2 "" H 3420 3160 60  0001 C CNN
@@
 	4070 4110 4170 4110
 $Comp
-L GND #PWR?
+L GND #PWR3
 U 1 1 5514565E
 P 4170 4610
-F 0 "#PWR?" H 4220 4660 60  0001 C CNN
+F 0 "#PWR3" H 4220 4660 60  0001 C CNN
 F 1 "GND" H 4170 4610 60  0001 C CNN
 F 2 "" H 4170 4610 60  0001 C CNN
@@
 $EndComp
 $Comp
-L GND #PWR?
+L GND #PWR8
 U 1 1 5514567E
 P 7370 4610
-F 0 "#PWR?" H 7420 4660 60  0001 C CNN
+F 0 "#PWR8" H 7420 4660 60  0001 C CNN
 F 1 "GND" H 7370 4610 60  0001 C CNN
 F 2 "" H 7370 4610 60  0001 C CNN
@@
 	4170 4310 4170 4610
 Wire Wire Line
-	2770 2860 2770 3360
+	2770 2860 2770 3010
+Wire Wire Line
+	2770 3010 2770 3260
+Wire Wire Line
+	2770 3260 2770 3360
 Wire Wire Line
 	2770 3010 2920 3010
@@
 Connection ~ 2770 3260
 $Comp
-L LD1117S33TR U?
+L LD1117S33TR U1
 U 1 1 55225E70
 P 1690 2910
-F 0 "U?" H 1690 3160 40  0000 C CNN
+F 0 "U1" H 1690 3160 40  0000 C CNN
 F 1 "LD1117S33TR" H 1690 3110 40  0000 C CNN
 F 2 "SOT-223" H 1690 3010 40  0000 C CNN
@@
 $EndComp
 Wire Wire Line
-	2090 2860 2770 2860
-$Comp
-L GND #PWR?
+	2090 2860 2320 2860
+Wire Wire Line
+	2320 2860 2770 2860
+$Comp
+L GND #PWR2
 U 1 1 552260D6
 P 1690 3350
-F 0 "#PWR?" H 1690 3100 50  0001 C CNN
+F 0 "#PWR2" H 1690 3100 50  0001 C CNN
 F 1 "GND" H 1690 3200 50  0000 C CNN
 F 2 "" H 1690 3350 60  0000 C CNN
@@
 	1690 3350 1690 3160
 $Comp
-L VCC #PWR?
+L VCC #PWR1
 U 1 1 55226122
 P 1200 2720
-F 0 "#PWR?" H 1200 2570 50  0001 C CNN
+F 0 "#PWR1" H 1200 2570 50  0001 C CNN
 F 1 "VCC" H 1200 2870 50  0000 C CNN
 F 2 "" H 1200 2720 60  0000 C CNN
@@
 Wire Wire Line
 	1200 2860 1290 2860
-$Comp
-L CP C?
-U 1 1 5522616D
-P 1200 3080
-F 0 "C?" H 1225 3180 50  0000 L CNN
-F 1 "CP" H 1225 2980 50  0000 L CNN
-F 2 "" H 1238 2930 30  0000 C CNN
-F 3 "" H 1200 3080 60  0000 C CNN
-	1    1200 3080
-	1    0    0    -1
-$EndComp
-$Comp
-L CP C?
-U 1 1 55226206
-P 2320 3110
-F 0 "C?" H 2345 3210 50  0000 L CNN
-F 1 "CP" H 2345 3010 50  0000 L CNN
-F 2 "" H 2358 2960 30  0000 C CNN
-F 3 "" H 2320 3110 60  0000 C CNN
-	1    2320 3110
-	1    0    0    -1
-$EndComp
-Wire Wire Line
-	1200 3230 1200 3310
-Wire Wire Line
-	1200 3310 2620 3310
-Wire Wire Line
-	2320 3310 2320 3260
-Wire Wire Line
-	1200 2720 1200 2930
+Wire Wire Line
+	1200 3170 1200 3310
+Wire Wire Line
+	1200 3310 2320 3310
+Wire Wire Line
+	2320 3310 2620 3310
+Wire Wire Line
+	2320 3310 2320 3170
+Wire Wire Line
+	1200 2720 1200 2860
+Wire Wire Line
+	1200 2860 1200 2970
 Connection ~ 1200 2860
 Wire Wire Line
-	2320 2960 2320 2860
+	2320 2970 2320 2860
 Connection ~ 2320 2860
 Wire Wire Line
 	2620 3310 2620 3110
 Connection ~ 2320 3310
+$Comp
+L CP_Small C1
+U 1 1 5522631D
+P 1200 3070
+F 0 "C1" H 1210 3140 50  0000 L CNN
+F 1 "10nF" H 1210 2990 50  0000 L CNN
+F 2 "" H 1200 3070 60  0000 C CNN
+F 3 "" H 1200 3070 60  0000 C CNN
+	1    1200 3070
+	1    0    0    -1
+$EndComp
+$Comp
+L CP_Small C2
+U 1 1 5522642C
+P 2320 3070
+F 0 "C2" H 2330 3140 50  0000 L CNN
+F 1 "10uF" H 2330 2990 50  0000 L CNN
+F 2 "" H 2320 3070 60  0000 C CNN
+F 3 "" H 2320 3070 60  0000 C CNN
+	1    2320 3070
+	1    0    0    -1
+$EndComp
 $EndSCHEMATC
